File: project-chibi-test-board.kicad_pcb (KiCad board)
At the start: 4 copper layers, 104.1 x 134.6 mm, 221 parts, among them J1 Conn_01x04, J10 Conn_01x02, J11 Conn_01x02, J12 Conn_02x06_Top_Bottom, J13 Conn_02x06_Top_Bottom, J14 Conn_02x06_Top_Bottom, J15 Conn_02x06_Top_Bottom, J16 Conn_01x02, J17 Conn_01x02, J18 Conn_Coaxial, J19 Conn_Coaxial, J2 Conn_Coaxial, J20 Conn_01x03, J21 Conn_01x03, J22 Conn_01x04, J23 USB_B_Micro, J24 Conn_01x06, J25 Conn_01x04, J26 Conn_Coaxial, J27 Conn_Coaxial, J28 Conn_01x03, J29 Conn_01x03, J3 Conn_Coaxial, J30 Conn_01x02, J31 Conn_01x02, J32 Conn_02x06_Top_Bottom, J33 Conn_02x06_Top_Bottom, J34 Conn_02x06_Top_Bottom, J35 Conn_02x06_Top_Bottom, J36 Conn_02x06_Top_Bottom, J37 Conn_02x06_Top_Bottom, J38 Conn_02x06_Top_Bottom, J39 Conn_02x06_Top_Bottom, J4 Conn_01x03, J40 Conn_01x02, J41 Conn_01x02, J42 Conn_Coaxial, J43 Conn_Coaxial, J44 Conn_01x04, J45 Conn_01x03, J46 Conn_01x03, J47 Conn_01x06, J5 Conn_01x03, J6 Conn_02x06_Top_Bottom, J7 Conn_02x06_Top_Bottom, J8 Conn_02x06_Top_Bottom, J9 Conn_01x06, SW1 SW_DIP_x08, SW2 SW_DIP_x08, U1 40 MHz, U10 5M240ZT144C5N, U11 5M1270ZF256C5N, U2 2.048 MHz, U3 5M40ZE64C5N, U4 5M2210ZF256C5N, U5 93LC56BT-OT, U6 5M240ZT144C5N, U7 LM1117-3.3, U8 LM1117-1.8, U9 FT232H, Y1 12 MHz

Commit message: add gnd test points
Parts:
- added J48: Conn_01x02, Connector_PinHeader_2.54mm:PinHeader_1x02_P2.54mm_Vertical, F.Cu at (108.5, 155.6)
- added J49: Conn_01x02, Connector_PinHeader_2.54mm:PinHeader_1x02_P2.54mm_Vertical, F.Cu at (128.3, 132.0)
- added J50: Conn_01x02, Connector_PinHeader_2.54mm:PinHeader_1x02_P2.54mm_Vertical, F.Cu at (132.6, 98.7)
- added J51: Conn_01x02, Connector_PinHeader_2.54mm:PinHeader_1x02_P2.54mm_Vertical, F.Cu at (100.2, 72.8)
- added J52: Conn_01x02, Connector_PinHeader_2.54mm:PinHeader_1x02_P2.54mm_Vertical, F.Cu at (87.0, 118.2)
- moved C1 31.3 mm to (85.6, 137.9)
- moved C2 31.3 mm to (87.5, 137.9)
- moved R1 31.3 mm to (83.7, 137.9)
- moved R2 31.3 mm to (81.8, 137.9)
- moved U1 31.3 mm to (86.5, 140.1)
- moved U2 31.3 mm to (82.4, 140.1)
- moved C41 0.64 mm to (73.9, 126.7)
- moved C47 0.64 mm to (73.6, 127.7)
- moved C54 0.64 mm to (74.6, 126.7)
- moved L3 0.64 mm to (73.1, 129.5)
Routing:
- net Net-(J23-Pad1): track 6.83 -> 0.00 mm
Other:
- net class USB added: clearance 0.1524, trace_width 0.1524, via_dia 0.6096, via_drill 0.3048

Commit message: rough 50z routing
Parts:
- moved J5 11.0 mm to (78.7, 81.3)
- moved J28 8.89 mm to (94.6, 165.7)
- moved J29 8.89 mm to (94.6, 154.3)
- moved J20 8.25 mm to (117.5, 73.7)
- moved J21 8.25 mm to (117.5, 85.1)
- moved J45 8.25 mm to (137.8, 147.3)
- moved J46 8.25 mm to (128.9, 147.3)
- moved J4 7.24 mm to (69.8, 81.3)
- moved J1 6.63 mm to (88.3, 68.6)
- moved D2 6.08 mm to (84.3, 67.9)
- moved R4 5.92 mm to (81.8, 67.9)
- moved D4 4.42 mm to (84.3, 71.8)
- moved R6 4.20 mm to (81.8, 71.8)
- moved D3 4.06 mm to (84.3, 69.8)
- moved D9 4.03 mm to (84.3, 75.6)
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Connections:
- net Net-(J2-Pad1) renamed /tgt-4x6/CLKIN0
- net Net-(J3-Pad1) renamed /tgt-4x6/CLKIN1
- U3 pad 1: /tgt-4x6/EXPAND0_4 -> /tgt-4x6/EXPAND0_0
- U3 pad 51: /tgt-4x6/EXPAND1_2 -> /tgt-4x6/EXPAND1_6
- U3 pad 52: /tgt-4x6/EXPAND1_6 -> /tgt-4x6/EXPAND1_2
- U3 pad 53: /tgt-4x6/EXPAND1_1 -> /tgt-4x6/EXPAND1_5
- U3 pad 54: /tgt-4x6/EXPAND1_5 -> /tgt-4x6/EXPAND1_1
- U3 pad 55: /tgt-4x6/EXPAND1_0 -> /tgt-4x6/EXPAND1_4
- U3 pad 56: /tgt-4x6/EXPAND1_4 -> /tgt-4x6/EXPAND1_0
- U3 pad 58: /tgt-4x6/EXPAND0_3 -> /tgt-4x6/EXPAND0_7
- U3 pad 59: /tgt-4x6/EXPAND0_7 -> /tgt-4x6/EXPAND0_3
- U3 pad 60: /tgt-4x6/EXPAND0_2 -> /tgt-4x6/EXPAND0_6
- U3 pad 61: /tgt-4x6/EXPAND0_6 -> /tgt-4x6/EXPAND0_2
- U3 pad 62: /tgt-4x6/EXPAND0_1 -> /tgt-4x6/EXPAND0_5
- U3 pad 63: /tgt-4x6/EXPAND0_5 -> /tgt-4x6/EXPAND0_1
- U3 pad 64: /tgt-4x6/EXPAND0_0 -> /tgt-4x6/EXPAND0_4
Routing:
- net /tgt-4x6/EXPAND3_0: track 0.00 -> 31.4 mm
- net /tgt-4x6/EXPAND3_1: track 0.00 -> 28.7 mm
- net /tgt-4x6/EXPAND3_2: track 0.00 -> 26.0 mm
- net /tgt-4x6/EXPAND2_3: track 0.00 -> 24.6 mm
- net /tgt-4x6/EXPAND2_2: track 0.00 -> 24.2 mm
- net /tgt-4x6/EXPAND3_3: track 0.00 -> 23.3 mm
- net /tgt-4x6/EXPAND2_1: track 0.00 -> 22.7 mm, vias 0 -> 1
- net /tgt-4x6/EXPAND2_7: track 0.00 -> 22.5 mm
- net /tgt-4x6/EXPAND2_6: track 0.00 -> 22.1 mm
- net Net-(J1-Pad3): track 0.00 -> 21.6 mm
- net /tgt-4x6/EXPAND2_0: track 0.00 -> 20.8 mm, vias 0 -> 1
- net Net-(J1-Pad2): track 0.00 -> 20.0 mm
- net /tgt-4x6/EXPAND2_5: track 0.00 -> 20.0 mm, vias 0 -> 1
- net /tgt-4x6/EXPAND2_4: track 0.00 -> 18.8 mm, vias 0 -> 1
- net /tgt-4x6/CLKIN1: track 0.00 -> 18.5 mm
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Other:
- net class 50ohm added: clearance 0.1524, trace_width 0.3302, via_dia 0.6096, via_drill 0.3048

Commit message: rough 240z routing
Parts:
- moved J25 8.13 mm to (94.6, 142.9), turned to 90 degrees
- moved J48 6.50 mm to (109.9, 161.9)
- moved R20 0.89 mm to (71.1, 137.6)
- moved D11 0.89 mm to (71.1, 140.4)
Connections:
- net Net-(J26-Pad1) renamed /tgt-7x12/CLKIN0
- net Net-(J27-Pad1) renamed /tgt-7x12/CLKIN1
- U10 pad 141: /tgt-7x12/EXPAND3_1 -> /tgt-7x12/EXPAND3_5
- U10 pad 142: /tgt-7x12/EXPAND3_5 -> /tgt-7x12/EXPAND3_1
- U10 pad 143: /tgt-7x12/EXPAND3_0 -> /tgt-7x12/EXPAND3_4
- U10 pad 144: /tgt-7x12/EXPAND3_4 -> /tgt-7x12/EXPAND3_0
- U10 pad 31: /tgt-7x12/EXPAND1_3 -> /tgt-7x12/EXPAND1_7
- U10 pad 32: /tgt-7x12/EXPAND1_7 -> /tgt-7x12/EXPAND1_3
- U10 pad 5: /tgt-7x12/EXPAND0_1 -> /tgt-7x12/EXPAND0_5
- U10 pad 6: /tgt-7x12/EXPAND0_5 -> /tgt-7x12/EXPAND0_1
Routing:
- net /tgt-7x12/CLKIN1: track 0.00 -> 37.9 mm, vias 0 -> 1
- net /tgt-7x12/CLKIN0: track 0.00 -> 28.7 mm, vias 0 -> 1
- net Net-(J25-Pad3): track 0.00 -> 18.3 mm
- net /tgt-7x12/EXPAND1_0: track 0.00 -> 17.3 mm
- net Net-(J25-Pad2): track 0.00 -> 16.8 mm
- net /tgt-7x12/EXPAND2_3: track 0.00 -> 15.8 mm
- net /tgt-7x12/EXPAND1_1: track 0.00 -> 14.6 mm
- net /tgt-7x12/EXPAND2_7: track 0.00 -> 14.2 mm
- net /tgt-7x12/EXPAND2_2: track 0.00 -> 13.8 mm
- net /tgt-7x12/EXPAND1_4: track 0.00 -> 13.1 mm
- net /tgt-7x12/EXPAND1_3: track 0.00 -> 12.4 mm
- net /tgt-7x12/EXPAND1_2: track 0.00 -> 12.2 mm
- net /tgt-7x12/EXPAND2_6: track 0.00 -> 11.7 mm
- net /tgt-7x12/EXPAND2_1: track 0.00 -> 11.7 mm
- net /tgt-7x12/EXPAND1_5: track 0.00 -> 10.4 mm
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
Commit message: rough 1270z routing
Parts:
- moved C103 11.1 mm to (129.5, 166.8)
- moved J49 5.08 mm to (123.2, 132.0)
- moved J43 5.08 mm to (121.3, 141.6)
- moved J46 5.08 mm to (123.8, 147.3)
- moved J42 5.08 mm to (130.2, 141.6)
- moved J45 5.08 mm to (132.7, 147.3)
- moved R31 3.71 mm to (115.7, 165.1)
- moved R28 3.50 mm to (115.7, 166.4)
- moved D22 2.94 mm to (112.2, 166.4)
- moved D19 2.79 mm to (112.2, 165.1)
- moved D20 2.66 mm to (112.2, 163.8)
- moved D21 2.55 mm to (112.2, 167.6)
- moved R29 2.47 mm to (115.7, 163.8)
- moved R30 2.34 mm to (115.7, 167.6)
- moved D12 1.91 mm to (112.7, 161.0)
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Connections:
- U11 pad A2: /tgt-10x16/EXPAND1_6 -> /tgt-10x16/EXPAND0_4
- U11 pad B1: /tgt-10x16/EXPAND1_1 -> /tgt-10x16/EXPAND1_3
- U11 pad B3: /tgt-10x16/EXPAND1_4 -> /tgt-10x16/EXPAND0_1
- U11 pad B4: /tgt-10x16/EXPAND1_7 -> /tgt-10x16/EXPAND0_2
- U11 pad C14: /tgt-10x16/EXPAND2_2 -> /tgt-10x16/EXPAND2_1
- U11 pad C15: /tgt-10x16/EXPAND2_4 -> /tgt-10x16/EXPAND2_5
- U11 pad C2: /tgt-10x16/EXPAND0_1 -> /tgt-10x16/EXPAND1_7
- U11 pad C3: /tgt-10x16/EXPAND0_3 -> /tgt-10x16/EXPAND0_0
- U11 pad C5: /tgt-10x16/EXPAND1_5 -> /tgt-10x16/EXPAND0_6
- U11 pad C6: /tgt-10x16/EXPAND1_3 -> /tgt-10x16/EXPAND0_7
- U11 pad D1: /tgt-10x16/EXPAND0_7 -> /tgt-10x16/EXPAND1_1
- U11 pad D13: /tgt-10x16/EXPAND2_0 -> /tgt-10x16/EXPAND2_4
- U11 pad D14: /tgt-10x16/EXPAND2_6 -> /tgt-10x16/EXPAND2_2
- U11 pad D2: /tgt-10x16/EXPAND0_5 -> /tgt-10x16/EXPAND1_6
- U11 pad D3: /tgt-10x16/EXPAND0_0 -> /tgt-10x16/EXPAND1_2
- U11 pad D4: /tgt-10x16/EXPAND1_2 -> /tgt-10x16/EXPAND0_5
- U11 pad D5: /tgt-10x16/EXPAND1_0 -> /tgt-10x16/EXPAND0_3
- U11 pad E12: /tgt-10x16/EXPAND2_5 -> /tgt-10x16/EXPAND2_0
- U11 pad E14: /tgt-10x16/EXPAND2_1 -> /tgt-10x16/EXPAND2_6
- U11 pad E3: /tgt-10x16/EXPAND0_2 -> /tgt-10x16/EXPAND1_5
- U11 pad E4: /tgt-10x16/EXPAND0_4 -> /tgt-10x16/EXPAND1_0
- U11 pad E5: /tgt-10x16/EXPAND0_6 -> /tgt-10x16/EXPAND1_4
- U11 pad K1: Net-(U11-PadK1) -> /tgt-10x16/ADBUS0
- U11 pad K2: Net-(U11-PadK2) -> /tgt-10x16/ADBUS1
- U11 pad K3: Net-(U11-PadK3) -> /tgt-10x16/ACBUS0
- U11 pad K4: Net-(U11-PadK4) -> /tgt-10x16/ACBUS4
- U11 pad L1: Net-(U11-PadL1) -> /tgt-10x16/ADBUS2
- U11 pad L11: /tgt-10x16/ADBUS1 -> Net-(U11-PadL11)
- U11 pad L12: /tgt-10x16/ADBUS3 -> Net-(U11-PadL12)
- U11 pad L13: /tgt-10x16/ADBUS5 -> Net-(U11-PadL13)
- U11 pad L14: /tgt-10x16/ADBUS7 -> Net-(U11-PadL14)
- U11 pad L15: /tgt-10x16/ADBUS0 -> Net-(U11-PadL15)
- U11 pad L2: Net-(U11-PadL2) -> /tgt-10x16/ADBUS3
- U11 pad L3: Net-(U11-PadL3) -> /tgt-10x16/ACBUS1
- U11 pad L4: Net-(U11-PadL4) -> /tgt-10x16/ACBUS5
- U11 pad M1: Net-(U11-PadM1) -> /tgt-10x16/ADBUS4
- U11 pad M13: /tgt-10x16/ACBUS1 -> Net-(U11-PadM13)
- U11 pad M14: /tgt-10x16/ACBUS3 -> Net-(U11-PadM14)
- U11 pad M15: /tgt-10x16/ADBUS4 -> Net-(U11-PadM15)
- U11 pad M16: /tgt-10x16/ADBUS2 -> Net-(U11-PadM16)
- U11 pad M2: Net-(U11-PadM2) -> /tgt-10x16/ADBUS5
- U11 pad M3: Net-(U11-PadM3) -> /tgt-10x16/ACBUS2
- U11 pad M4: Net-(U11-PadM4) -> /tgt-10x16/ACBUS6
- U11 pad N1: Net-(U11-PadN1) -> /tgt-10x16/ADBUS6
- U11 pad N13: /tgt-10x16/ACBUS5 -> Net-(U11-PadN13)
- U11 pad N14: /tgt-10x16/ACBUS2 -> Net-(U11-PadN14)
- U11 pad N15: /tgt-10x16/ACBUS0 -> Net-(U11-PadN15)
- U11 pad N16: /tgt-10x16/ADBUS6 -> Net-(U11-PadN16)
- U11 pad N2: Net-(U11-PadN2) -> /tgt-10x16/ADBUS7
- U11 pad N3: Net-(U11-PadN3) -> /tgt-10x16/ACBUS3
- U11 pad N5: /tgt-10x16/EXPAND3_3 -> /tgt-10x16/EXPAND3_4
- U11 pad N6: /tgt-10x16/EXPAND3_6 -> /tgt-10x16/EXPAND3_0
- U11 pad P14: /tgt-10x16/ACBUS6 -> Net-(U11-PadP14)
- U11 pad P15: /tgt-10x16/ACBUS4 -> Net-(U11-PadP15)
- U11 pad P4: /tgt-10x16/EXPAND3_1 -> /tgt-10x16/EXPAND3_5
- U11 pad P5: /tgt-10x16/EXPAND3_5 -> /tgt-10x16/EXPAND3_1
- U11 pad R1: /tgt-10x16/EXPAND3_0 -> /tgt-10x16/EXPAND3_7
- U11 pad R3: /tgt-10x16/EXPAND3_2 -> /tgt-10x16/EXPAND3_6
- U11 pad R4: /tgt-10x16/EXPAND3_7 -> /tgt-10x16/EXPAND3_2
- U11 pad T2: /tgt-10x16/EXPAND3_4 -> /tgt-10x16/EXPAND3_3
Routing:
- net /tgt-10x16/EXPAND1_0: track 0.00 -> 30.0 mm, vias 0 -> 2
- net /tgt-10x16/EXPAND1_4: track 0.00 -> 29.2 mm
- net /tgt-10x16/EXPAND3_3: track 0.00 -> 28.0 mm
- net /tgt-10x16/EXPAND3_7: track 0.00 -> 28.0 mm
- net /tgt-10x16/EXPAND3_2: track 0.00 -> 27.0 mm
- net /tgt-10x16/EXPAND1_5: track 0.00 -> 25.1 mm
- net /tgt-10x16/EXPAND1_1: track 0.00 -> 24.8 mm
- net /tgt-10x16/EXPAND1_2: track 0.00 -> 24.5 mm, vias 0 -> 2
- net /tgt-10x16/EXPAND3_6: track 0.00 -> 24.5 mm
- net /tgt-10x16/EXPAND3_1: track 0.00 -> 23.7 mm
- net /tgt-10x16/EXPAND3_5: track 0.00 -> 22.8 mm, vias 0 -> 2
- net /tgt-10x16/EXPAND3_0: track 0.00 -> 22.2 mm
- net Net-(J44-Pad3): track 0.00 -> 22.2 mm, vias 0 -> 2
- net /tgt-10x16/EXPAND1_6: track 0.00 -> 21.8 mm
- net /tgt-10x16/CLK1: track 0.00 -> 21.5 mm
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
Commit message: rough 2240z routing
Parts:
- moved J18 27.3 mm to (124.5, 95.2)
- moved R22 25.6 mm to (102.3, 125.2)
- moved R23 25.6 mm to (102.3, 123.7)
- moved D13 25.6 mm to (105.0, 125.2)
- moved D14 25.6 mm to (105.0, 123.7)
- moved J22 18.1 mm to (113.7, 73.0), turned to 270 degrees
- moved J20 18.0 mm to (127.0, 88.9), turned to 270 degrees
- moved J47 9.94 mm to (117.5, 101.6), turned to 90 degrees
- moved C99 9.71 mm to (129.5, 81.5)
- moved J50 3.14 mm to (135.3, 100.3)
- moved R19 1.15 mm to (136.5, 89.0)
- moved D10 1.14 mm to (136.5, 91.7)
- moved J19 0.64 mm to (111.1, 82.5)
- moved J2 0.63 mm to (72.4, 87.6)
- moved J3 0.63 mm to (81.3, 87.6)
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Connections:
- U11 pad B1: /tgt-10x16/EXPAND1_3 -> /tgt-10x16/EXPAND1_7
- U11 pad C2: /tgt-10x16/EXPAND1_7 -> /tgt-10x16/EXPAND1_3
- U11 pad D1: /tgt-10x16/EXPAND1_1 -> /tgt-10x16/EXPAND1_5
- U11 pad D2: /tgt-10x16/EXPAND1_6 -> /tgt-10x16/EXPAND1_2
- U11 pad D3: /tgt-10x16/EXPAND1_2 -> /tgt-10x16/EXPAND1_6
- U11 pad E3: /tgt-10x16/EXPAND1_5 -> /tgt-10x16/EXPAND1_1
- U11 pad E4: /tgt-10x16/EXPAND1_0 -> /tgt-10x16/EXPAND1_4
- U11 pad E5: /tgt-10x16/EXPAND1_4 -> /tgt-10x16/EXPAND1_0
- U4 pad B1: /tgt-13x20/EXPAND1_1 -> /tgt-13x20/EXPAND0_7
- U4 pad B3: /tgt-13x20/EXPAND1_6 -> /tgt-13x20/EXPAND1_4
- U4 pad C14: /tgt-13x20/EXPAND2_2 -> /tgt-13x20/EXPAND2_1
- U4 pad C15: /tgt-13x20/EXPAND2_3 -> /tgt-13x20/EXPAND2_2
- U4 pad C2: /tgt-13x20/EXPAND0_1 -> /tgt-13x20/EXPAND0_3
- U4 pad C3: /tgt-13x20/EXPAND0_2 -> /tgt-13x20/EXPAND1_1
- U4 pad C4: /tgt-13x20/EXPAND1_4 -> /tgt-13x20/EXPAND1_5
- U4 pad C5: /tgt-13x20/EXPAND1_5 -> /tgt-13x20/EXPAND1_2
- U4 pad D1: /tgt-13x20/EXPAND0_6 -> /tgt-13x20/EXPAND0_1
- U4 pad D13: /tgt-13x20/EXPAND2_0 -> /tgt-13x20/EXPAND2_4
- U4 pad D15: /tgt-13x20/EXPAND2_7 -> /tgt-13x20/EXPAND2_6
- U4 pad D2: /tgt-13x20/EXPAND0_4 -> /tgt-13x20/EXPAND0_2
- U4 pad D3: /tgt-13x20/EXPAND0_0 -> /tgt-13x20/EXPAND0_6
- U4 pad D4: /tgt-13x20/EXPAND1_2 -> /tgt-13x20/EXPAND1_6
- U4 pad D5: /tgt-13x20/EXPAND1_3 -> /tgt-13x20/EXPAND1_7
- U4 pad D6: /tgt-13x20/EXPAND1_7 -> /tgt-13x20/EXPAND1_3
- U4 pad E12: /tgt-13x20/EXPAND2_6 -> /tgt-13x20/EXPAND2_7
- U4 pad E13: /tgt-13x20/EXPAND2_4 -> /tgt-13x20/EXPAND2_0
- U4 pad E14: /tgt-13x20/EXPAND2_1 -> /tgt-13x20/EXPAND2_3
- U4 pad E3: /tgt-13x20/EXPAND0_3 -> /tgt-13x20/EXPAND0_4
- U4 pad E5: /tgt-13x20/EXPAND0_7 -> /tgt-13x20/EXPAND0_0
- U4 pad L11: /tgt-13x20/ADBUS0 -> Net-(U4-PadL11)
- U4 pad L12: /tgt-13x20/ADBUS2 -> Net-(U4-PadL12)
- U4 pad L13: /tgt-13x20/ADBUS4 -> Net-(U4-PadL13)
- U4 pad L14: /tgt-13x20/ADBUS6 -> Net-(U4-PadL14)
- U4 pad L15: /tgt-13x20/ADBUS1 -> /tgt-13x20/ADBUS0
- U4 pad M13: /tgt-13x20/ACBUS0 -> Net-(U4-PadM13)
- U4 pad M14: /tgt-13x20/ACBUS2 -> Net-(U4-PadM14)
- U4 pad M15: /tgt-13x20/ADBUS5 -> /tgt-13x20/ADBUS2
- U4 pad M16: /tgt-13x20/ADBUS3 -> /tgt-13x20/ADBUS1
- U4 pad N13: /tgt-13x20/ACBUS4 -> Net-(U4-PadN13)
- U4 pad N14: /tgt-13x20/ACBUS3 -> Net-(U4-PadN14)
- U4 pad N15: /tgt-13x20/ACBUS1 -> /tgt-13x20/ADBUS4
- U4 pad N16: /tgt-13x20/ADBUS7 -> /tgt-13x20/ADBUS3
- U4 pad N5: /tgt-13x20/EXPAND3_2 -> /tgt-13x20/EXPAND3_4
- U4 pad N6: /tgt-13x20/EXPAND3_7 -> /tgt-13x20/EXPAND3_0
- U4 pad P14: /tgt-13x20/ACBUS6 -> Net-(U4-PadP14)
- U4 pad P15: /tgt-13x20/ACBUS5 -> /tgt-13x20/ADBUS5
- U4 pad P4: /tgt-13x20/EXPAND3_0 -> /tgt-13x20/EXPAND3_7
- U4 pad P5: /tgt-13x20/EXPAND3_4 -> /tgt-13x20/EXPAND3_1
- U4 pad R1: /tgt-13x20/EXPAND3_1 -> /tgt-13x20/EXPAND3_3
- U4 pad R11: Net-(U4-PadR11) -> /tgt-13x20/ACBUS6
- U4 pad R12: Net-(U4-PadR12) -> /tgt-13x20/ACBUS4
- U4 pad R13: Net-(U4-PadR13) -> /tgt-13x20/ACBUS2
- U4 pad R14: Net-(U4-PadR14) -> /tgt-13x20/ACBUS0
- U4 pad R16: Net-(U4-PadR16) -> /tgt-13x20/ADBUS7
- U4 pad R3: /tgt-13x20/EXPAND3_3 -> /tgt-13x20/EXPAND3_2
- U4 pad R4: /tgt-13x20/EXPAND3_6 -> /tgt-13x20/EXPAND3_5
- U4 pad T11: Net-(U4-PadT11) -> /tgt-13x20/ACBUS5
- U4 pad T12: Net-(U4-PadT12) -> /tgt-13x20/ACBUS3
- U4 pad T13: Net-(U4-PadT13) -> /tgt-13x20/ACBUS1
- U4 pad T15: Net-(U4-PadT15) -> /tgt-13x20/ADBUS6
- U4 pad T2: /tgt-13x20/EXPAND3_5 -> /tgt-13x20/EXPAND3_6
Routing:
- net /tgt-13x20/CLK1: track 0.00 -> 38.9 mm, vias 0 -> 1
- net /tgt-13x20/CLK0: track 0.00 -> 35.6 mm, vias 0 -> 1
- net /tgt-13x20/EXPAND3_0: track 0.00 -> 30.0 mm
- net /tgt-13x20/EXPAND2_7: track 0.00 -> 26.5 mm
- net /tgt-13x20/EXPAND3_1: track 0.00 -> 24.8 mm
- net /tgt-13x20/EXPAND3_4: track 0.00 -> 24.7 mm
- net /tgt-13x20/EXPAND2_3: track 0.00 -> 24.7 mm
- net /tgt-13x20/EXPAND2_2: track 0.00 -> 21.3 mm
- net /tgt-13x20/EXPAND2_1: track 0.00 -> 20.3 mm
- net /tgt-13x20/EXPAND2_6: track 0.00 -> 20.3 mm
- net /tgt-13x20/EXPAND2_0: track 0.00 -> 20.2 mm
- net /tgt-13x20/EXPAND3_2: track 0.00 -> 20.0 mm
- net Net-(J22-Pad3): track 0.00 -> 19.1 mm
- net /tgt-13x20/EXPAND3_5: track 0.00 -> 19.0 mm
- net /tgt-13x20/EXPAND2_5: track 0.00 -> 18.4 mm
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